Commit message: V0 four-bar knee drive (V1 dims); move SpotMicro ref to references/
- URDF: 60 mm femur/tibia, crank+coupler four-bar, loop constraint in sim
- LegConfig L2/L3 = 60 mm; test_stand sliders: hip_abduction, hip_flexion, knee_drive
- Move spot-micro/ → references/spot-micro/; update README paths and leg docs

Co-authored-by: Cursor <cursoragent@cursor.com>

File: V0_test_stand/urdf/leg_test_stand.urdf (robot description, URDF)
Before this commit: robot spot_micro_leg_test_stand, 5 links, 4 joints
Links:
- removed link lower_leg_link
- removed link upper_leg_link
- added link coupler_link, mass 0.05; collision cylinder length=0.060 radius=0.006; visual cylinder length=0.060 radius=0.006
- added link crank_link, mass 0.04; collision cylinder length=0.029 radius=0.007; visual cylinder length=0.029 radius=0.007
- added link femur_link, mass 0.12; collision cylinder length=0.060 radius=0.010; visual cylinder length=0.060 radius=0.010
- added link tibia_link, mass 0.08; collision cylinder length=0.060 radius=0.008; visual cylinder length=0.060 radius=0.008
- link foot_link: geometry collision sphere radius=0.012; visual sphere radius=0.012
- link shoulder_link: mass 0.10 -> 0.15; geometry collision cylinder length=0.055 radius=0.012; visual box size=0.033 0.008 0.008
Joints:
- removed joint knee_flexion
- added joint coupler_passive: type revolute, parent crank_link, child coupler_link, origin xyz=0 0 -0.029 rpy=0 0 0, axis 0 1 0, limit lower=-3.14 upper=3.14 effort=0 velocity=10.0
- added joint knee_drive: type revolute, parent shoulder_link, child crank_link, origin xyz=-0.033 -0.055 0 rpy=0 0 0, axis 0 1 0, limit lower=-2.618 upper=2.618 effort=12 velocity=6.28
- added joint knee_passive: type revolute, parent femur_link, child tibia_link, origin xyz=0 0 -0.060 rpy=0 0 0, axis 0 1 0, limit lower=-2.618 upper=2.618 effort=0 velocity=10.0
- joint foot_fixed: origin xyz=0 0 -0.130 -> xyz=0 0 -0.060; parent lower_leg_link -> tibia_link
- joint hip_flexion: child upper_leg_link -> femur_link
